File: ErgoGrid-pcb/ErgoGrid-pcb.kicad_sch (KiCad schematic)
At the start: 61 parts, among them J1 MCU_inside, J10 Joystick_R, J2 MCU_outside, J3 USB_5V, J4 AudioJack4_L, J5 AudioJack4_R, J6 MCU_3pin, J7 Battery, J8 OLED, J9 Joystick_L, U1 DRV2667

Commit message: started PCB routing
Parts:
- added C1, C2: 100n, Capacitor_SMD:C_0805_2012Metric, symbol C_Small:C_Small
- added H1: Joystick_L, ErgoGrid:Joystick_nintendo_switch, symbol MountingHole_Pad_MP:MountingHole_Pad_MP
- added H2: Joystick_R, ErgoGrid:Joystick_nintendo_switch, symbol MountingHole_Pad_MP:MountingHole_Pad_MP
- added J2: Joystick_L2, Connector_FFC-FPC:Amphenol_F32Q-1A7x1-11005_1x05-1MP_P0.5mm_Horizontal, symbol Conn_01x05_MountingPin:Conn_01x05_MountingPin
- added J7: Joystick_R2, Connector_FFC-FPC:Amphenol_F32Q-1A7x1-11005_1x05-1MP_P0.5mm_Horizontal, symbol Conn_01x05_MountingPin:Conn_01x05_MountingPin
- J1: renamed from J9; value Joystick_L -> Joystick_L1
- J3: renamed from J6; symbol Conn_01x05:Conn_01x05 -> Conn_01x03:Conn_01x03
- J6: renamed from J10; value Joystick_R -> Joystick_R1
- JP1: renamed from JP32; value GND_bat_L -> GND_bat_R; footprint Jumper:SolderJumper-2_P1.3mm_Open_TrianglePad1.0x1.5mm -> ErgoGrid:SolderJumper
- JP10: renamed from JP13; value GND2_ins -> GND2_R; footprint Jumper:SolderJumper-2_P1.3mm_Open_TrianglePad1.0x1.5mm -> ErgoGrid:SolderJumper
- JP11: renamed from JP2; value RX_outs -> TX_R; footprint Jumper:SolderJumper-2_P1.3mm_Open_TrianglePad1.0x1.5mm -> ErgoGrid:SolderJumper
- JP12: renamed from JP14; value GND2_outs -> GND2_L; footprint Jumper:SolderJumper-2_P1.3mm_Open_TrianglePad1.0x1.5mm -> ErgoGrid:SolderJumper
- JP13: renamed from JP25; footprint Jumper:SolderJumper-2_P1.3mm_Open_TrianglePad1.0x1.5mm -> ErgoGrid:SolderJumper
- JP14: renamed from JP26; footprint Jumper:SolderJumper-2_P1.3mm_Open_TrianglePad1.0x1.5mm -> ErgoGrid:SolderJumper
- JP15: renamed from JP28; footprint Jumper:SolderJumper-2_P1.3mm_Open_TrianglePad1.0x1.5mm -> ErgoGrid:SolderJumper
- JP16: renamed from JP29; footprint Jumper:SolderJumper-2_P1.3mm_Open_TrianglePad1.0x1.5mm -> ErgoGrid:SolderJumper
- JP17: renamed from JP31; footprint Jumper:SolderJumper-2_P1.3mm_Open_TrianglePad1.0x1.5mm -> ErgoGrid:SolderJumper
- JP18: renamed from JP34; footprint Jumper:SolderJumper-2_P1.3mm_Open_TrianglePad1.0x1.5mm -> ErgoGrid:SolderJumper
- JP19: renamed from JP35; footprint Jumper:SolderJumper-2_P1.3mm_Open_TrianglePad1.0x1.5mm -> ErgoGrid:SolderJumper
- JP2: renamed from JP33; value GND_bat_R -> GND_bat_L; footprint Jumper:SolderJumper-2_P1.3mm_Open_TrianglePad1.0x1.5mm -> ErgoGrid:SolderJumper
- JP20: renamed from JP36; footprint Jumper:SolderJumper-2_P1.3mm_Open_TrianglePad1.0x1.5mm -> ErgoGrid:SolderJumper
- JP21: renamed from JP9; value GND3_ins -> GND3_L; footprint Jumper:SolderJumper-2_P1.3mm_Open_TrianglePad1.0x1.5mm -> ErgoGrid:SolderJumper
- JP22: renamed from JP21; value RST_ins -> RST_R; footprint Jumper:SolderJumper-2_P1.3mm_Open_TrianglePad1.0x1.5mm -> ErgoGrid:SolderJumper
- JP23: renamed from JP10; value GND3_outs -> GND3_R; footprint Jumper:SolderJumper-2_P1.3mm_Open_TrianglePad1.0x1.5mm -> ErgoGrid:SolderJumper
- JP24: renamed from JP22; value RST_outs -> RST_L; footprint Jumper:SolderJumper-2_P1.3mm_Open_TrianglePad1.0x1.5mm -> ErgoGrid:SolderJumper
- JP25: renamed from JP3; value GND4_ins -> GND4_L; footprint Jumper:SolderJumper-2_P1.3mm_Open_TrianglePad1.0x1.5mm -> ErgoGrid:SolderJumper
- JP26: renamed from JP15; value VCC_ins -> VCC_R; footprint Jumper:SolderJumper-2_P1.3mm_Open_TrianglePad1.0x1.5mm -> ErgoGrid:SolderJumper
- JP27: renamed from JP4; value GND4_outs -> GND4_R; footprint Jumper:SolderJumper-2_P1.3mm_Open_TrianglePad1.0x1.5mm -> ErgoGrid:SolderJumper
- JP28: renamed from JP16; value VCC_outs -> VCC_L; footprint Jumper:SolderJumper-2_P1.3mm_Open_TrianglePad1.0x1.5mm -> ErgoGrid:SolderJumper
- JP29: renamed from JP11; value SDA_ins -> SDA_L; footprint Jumper:SolderJumper-2_P1.3mm_Open_TrianglePad1.0x1.5mm -> ErgoGrid:SolderJumper
- JP3: renamed from JP27; value Plus_bat_L -> Plus_bat_R; footprint Jumper:SolderJumper-2_P1.3mm_Open_TrianglePad1.0x1.5mm -> ErgoGrid:SolderJumper
- JP30: renamed from JP23; value AIN0_ins -> AIN0_R; footprint Jumper:SolderJumper-2_P1.3mm_Open_TrianglePad1.0x1.5mm -> ErgoGrid:SolderJumper
- JP31: renamed from JP12; value SDA_outs -> SDA_R; footprint Jumper:SolderJumper-2_P1.3mm_Open_TrianglePad1.0x1.5mm -> ErgoGrid:SolderJumper
- JP32: renamed from JP24; value AIN0_outs -> AIN0_L; footprint Jumper:SolderJumper-2_P1.3mm_Open_TrianglePad1.0x1.5mm -> ErgoGrid:SolderJumper
- JP33: renamed from JP5; value SCL_ins -> SCL_L; footprint Jumper:SolderJumper-2_P1.3mm_Open_TrianglePad1.0x1.5mm -> ErgoGrid:SolderJumper
- JP34: renamed from JP17; value AIN1_ins -> AIN1_R; footprint Jumper:SolderJumper-2_P1.3mm_Open_TrianglePad1.0x1.5mm -> ErgoGrid:SolderJumper
- JP35: renamed from JP6; value SCL_outs -> SCL_R; footprint Jumper:SolderJumper-2_P1.3mm_Open_TrianglePad1.0x1.5mm -> ErgoGrid:SolderJumper
- JP36: renamed from JP18; value AIN1_outs -> AIN1_L; footprint Jumper:SolderJumper-2_P1.3mm_Open_TrianglePad1.0x1.5mm -> ErgoGrid:SolderJumper
- JP4: renamed from JP30; value Plus_bat_R -> Plus_bat_L; footprint Jumper:SolderJumper-2_P1.3mm_Open_TrianglePad1.0x1.5mm -> ErgoGrid:SolderJumper
- JP5: renamed from JP7; value TX_ins -> RX_L; footprint Jumper:SolderJumper-2_P1.3mm_Open_TrianglePad1.0x1.5mm -> ErgoGrid:SolderJumper
- JP6: renamed from JP19; value BAT_ins -> BAT_R; footprint Jumper:SolderJumper-2_P1.3mm_Open_TrianglePad1.0x1.5mm -> ErgoGrid:SolderJumper
- JP7: renamed from JP8; value TX_outs -> RX_R; footprint Jumper:SolderJumper-2_P1.3mm_Open_TrianglePad1.0x1.5mm -> ErgoGrid:SolderJumper
- JP8: renamed from JP20; value BAT_outs -> BAT_L; footprint Jumper:SolderJumper-2_P1.3mm_Open_TrianglePad1.0x1.5mm -> ErgoGrid:SolderJumper
- JP9: renamed from JP1; value RX_ins -> TX_L; footprint Jumper:SolderJumper-2_P1.3mm_Open_TrianglePad1.0x1.5mm -> ErgoGrid:SolderJumper
- S1: value RST_L -> RST_R; footprint Button_Switch_SMD:SW_SPST_EVQP7C -> ErgoGrid:ResetButton; symbol SW_Push:SW_Push -> SW_Push_Shielded:SW_Push_Shielded
- S2: value RST_R -> RST_L; footprint Button_Switch_SMD:SW_SPST_EVQP7C -> ErgoGrid:ResetButton; symbol SW_Push:SW_Push -> SW_Push_Shielded:SW_Push_Shielded
- renumbered C4 to C3, C1 to C4, C3 to C6, C2 to C7, J8 to J10, J4 to J11, J5 to J12, J1 to J4, J3 to J5, J2 to J8, J7 to J9, R3 to R1, R1 to R2, R2 to R3
Connections:
- net AIN_0: now also J2.2 (Pin_2), J7.2 (Pin_2)
- net AIN_1: now also J2.5 (Pin_5), J7.5 (Pin_5)
- net EncA: no longer J3.5 (Pin_5)
- net EncB: no longer J3.4 (Pin_4)
- net GND: now also S1.SH (B), S2.2, S2.SH (B), C1.1, C2.1, H1.MP, H2.MP, J2.4 (Pin_4), J2.MP (MountPin), J7.4 (Pin_4), J7.MP (MountPin); no longer S2.1
- net JoyBtn: now also J2.3 (Pin_3), J7.3 (Pin_3)
- net RST: now also S2.1; no longer S2.2
- net RX: now also JP5.2 (B), JP7.1 (A); no longer JP11.1 (A), JP9.2 (B)
- net TX: now also JP11.1 (A), JP9.2 (B); no longer JP5.2 (B), JP7.1 (A)
- net VCC: now also C1.2, C2.2, J2.1 (Pin_1), J7.1 (Pin_1)
Other:
- moved on the sheet: J1, J6
