File: ErgoGrid-pcb/key_grid.kicad_sch (KiCad schematic)
At the start: 69 parts, among them SW1 SW_Push, SW10 SW_Push, SW11 SW_Push, SW12 SW_Push, SW13 SW_Push, SW14 SW_Push, SW15 SW_Push, SW16 SW_Push, SW17 SW_Push, SW18 SW_Push, SW19 SW_Push, SW2 SW_Push, SW20 SW_Push, SW21 SW_Push, SW3 SW_Push, SW4 SW_Push, SW5 SW_Push, SW6 SW_Push, SW7 SW_Push, SW8 SW_Push, SW9 SW_Push

Commit message: started PCB routing
Parts:
- added C10, C11, C8, C9: 100n, Capacitor_SMD:C_0805_2012Metric, symbol C_Small:C_Small
- added D19: 1N4148W, Diode_SMD:D_SOD-123, symbol D_Small_Filled:D_Small_Filled
- added LD24: SK6812MINI, ErgoGrid:SK6812_mini-e_rgb_reversible, symbol SK6812:SK6812
- added SW19: SW_Push, keyswitches:Kailh_socket_PG1350_reversible, symbol SW_Push:SW_Push
- JP37: renamed from JP38; footprint Jumper:SolderJumper-2_P1.3mm_Open_TrianglePad1.0x1.5mm -> ErgoGrid:SolderJumper
- JP38: renamed from JP37; footprint Jumper:SolderJumper-2_P1.3mm_Open_TrianglePad1.0x1.5mm -> ErgoGrid:SolderJumper
- LD1: renamed from D1; footprint LED_SMD:LED_SK6812MINI-E_3.2x2.8mm_P1.5mm_ReverseMount -> ErgoGrid:SK6812_mini-e_rgb_reversible; symbol SK6812MINI:SK6812MINI -> SK6812:SK6812
- LD10: renamed from D4; footprint LED_SMD:LED_SK6812MINI-E_3.2x2.8mm_P1.5mm_ReverseMount -> ErgoGrid:SK6812_mini-e_rgb_reversible; symbol SK6812MINI:SK6812MINI -> SK6812:SK6812
- LD11: renamed from D10; footprint LED_SMD:LED_SK6812MINI-E_3.2x2.8mm_P1.5mm_ReverseMount -> ErgoGrid:SK6812_mini-e_rgb_reversible; symbol SK6812MINI:SK6812MINI -> SK6812:SK6812
- LD12: renamed from D16; footprint LED_SMD:LED_SK6812MINI-E_3.2x2.8mm_P1.5mm_ReverseMount -> ErgoGrid:SK6812_mini-e_rgb_reversible; symbol SK6812MINI:SK6812MINI -> SK6812:SK6812
- LD13: renamed from D5; footprint LED_SMD:LED_SK6812MINI-E_3.2x2.8mm_P1.5mm_ReverseMount -> ErgoGrid:SK6812_mini-e_rgb_reversible; symbol SK6812MINI:SK6812MINI -> SK6812:SK6812
- LD14: renamed from D11; footprint LED_SMD:LED_SK6812MINI-E_3.2x2.8mm_P1.5mm_ReverseMount -> ErgoGrid:SK6812_mini-e_rgb_reversible; symbol SK6812MINI:SK6812MINI -> SK6812:SK6812
- LD15: renamed from D17; footprint LED_SMD:LED_SK6812MINI-E_3.2x2.8mm_P1.5mm_ReverseMount -> ErgoGrid:SK6812_mini-e_rgb_reversible; symbol SK6812MINI:SK6812MINI -> SK6812:SK6812
- LD16: renamed from D19; footprint LED_SMD:LED_SK6812MINI-E_3.2x2.8mm_P1.5mm_ReverseMount -> ErgoGrid:SK6812_mini-e_rgb_reversible; symbol SK6812MINI:SK6812MINI -> SK6812:SK6812
- LD17: renamed from D6; footprint LED_SMD:LED_SK6812MINI-E_3.2x2.8mm_P1.5mm_ReverseMount -> ErgoGrid:SK6812_mini-e_rgb_reversible; symbol SK6812MINI:SK6812MINI -> SK6812:SK6812
- LD18: renamed from D12; footprint LED_SMD:LED_SK6812MINI-E_3.2x2.8mm_P1.5mm_ReverseMount -> ErgoGrid:SK6812_mini-e_rgb_reversible; symbol SK6812MINI:SK6812MINI -> SK6812:SK6812
- LD19: renamed from D18; footprint LED_SMD:LED_SK6812MINI-E_3.2x2.8mm_P1.5mm_ReverseMount -> ErgoGrid:SK6812_mini-e_rgb_reversible; symbol SK6812MINI:SK6812MINI -> SK6812:SK6812
- LD2: renamed from D7; footprint LED_SMD:LED_SK6812MINI-E_3.2x2.8mm_P1.5mm_ReverseMount -> ErgoGrid:SK6812_mini-e_rgb_reversible; symbol SK6812MINI:SK6812MINI -> SK6812:SK6812
- LD20: renamed from D20; footprint LED_SMD:LED_SK6812MINI-E_3.2x2.8mm_P1.5mm_ReverseMount -> ErgoGrid:SK6812_mini-e_rgb_reversible; symbol SK6812MINI:SK6812MINI -> SK6812:SK6812
- LD21: renamed from D23; footprint LED_SMD:LED_SK6812MINI-E_3.2x2.8mm_P1.5mm_ReverseMount -> ErgoGrid:SK6812_mini-e_rgb_reversible; symbol SK6812MINI:SK6812MINI -> SK6812:SK6812
- LD22: renamed from D22; footprint LED_SMD:LED_SK6812MINI-E_3.2x2.8mm_P1.5mm_ReverseMount -> ErgoGrid:SK6812_mini-e_rgb_reversible; symbol SK6812MINI:SK6812MINI -> SK6812:SK6812
- LD23: renamed from D21; footprint LED_SMD:LED_SK6812MINI-E_3.2x2.8mm_P1.5mm_ReverseMount -> ErgoGrid:SK6812_mini-e_rgb_reversible; symbol SK6812MINI:SK6812MINI -> SK6812:SK6812
- LD3: renamed from D13; footprint LED_SMD:LED_SK6812MINI-E_3.2x2.8mm_P1.5mm_ReverseMount -> ErgoGrid:SK6812_mini-e_rgb_reversible; symbol SK6812MINI:SK6812MINI -> SK6812:SK6812
- LD4: renamed from D2; footprint LED_SMD:LED_SK6812MINI-E_3.2x2.8mm_P1.5mm_ReverseMount -> ErgoGrid:SK6812_mini-e_rgb_reversible; symbol SK6812MINI:SK6812MINI -> SK6812:SK6812
- LD5: renamed from D8; footprint LED_SMD:LED_SK6812MINI-E_3.2x2.8mm_P1.5mm_ReverseMount -> ErgoGrid:SK6812_mini-e_rgb_reversible; symbol SK6812MINI:SK6812MINI -> SK6812:SK6812
- LD6: renamed from D14; footprint LED_SMD:LED_SK6812MINI-E_3.2x2.8mm_P1.5mm_ReverseMount -> ErgoGrid:SK6812_mini-e_rgb_reversible; symbol SK6812MINI:SK6812MINI -> SK6812:SK6812
- LD7: renamed from D3; footprint LED_SMD:LED_SK6812MINI-E_3.2x2.8mm_P1.5mm_ReverseMount -> ErgoGrid:SK6812_mini-e_rgb_reversible; symbol SK6812MINI:SK6812MINI -> SK6812:SK6812
- LD8: renamed from D9; footprint LED_SMD:LED_SK6812MINI-E_3.2x2.8mm_P1.5mm_ReverseMount -> ErgoGrid:SK6812_mini-e_rgb_reversible; symbol SK6812MINI:SK6812MINI -> SK6812:SK6812
- LD9: renamed from D15; footprint LED_SMD:LED_SK6812MINI-E_3.2x2.8mm_P1.5mm_ReverseMount -> ErgoGrid:SK6812_mini-e_rgb_reversible; symbol SK6812MINI:SK6812MINI -> SK6812:SK6812
- renumbered D24 to D1, D38 to D10, D43 to D11, D27 to D12, D33 to D13, D39 to D14, D44 to D15, D28 to D16, D34 to D17, D40 to D18, D30 to D2, D29 to D20, D35 to D21, D41 to D22, D45 to D23, D36 to D3, D25 to D4, D31 to D5, D37 to D6, D42 to D7, D26 to D8, D32 to D9, SW15 to SW10, SW20 to SW11, SW4 to SW12, SW10 to SW13, SW16 to SW14, SW21 to SW15, SW5 to SW16, SW11 to SW17, SW17 to SW18, SW7 to SW2, SW6 to SW20, SW12 to SW21, SW18 to SW22, SW13 to SW3, SW2 to SW4, SW8 to SW5, SW14 to SW6, SW19 to SW7, SW3 to SW8
Connections:
- net GND: now also LD1.1 (VSS), LD10.1 (VSS), LD11.1 (VSS), LD12.1 (VSS), LD13.1 (VSS), LD14.1 (VSS), LD15.1 (VSS), LD16.1 (VSS), LD17.1 (VSS), LD18.1 (VSS), LD19.1 (VSS), LD2.1 (VSS), LD20.1 (VSS), LD21.1 (VSS), LD22.1 (VSS), LD23.1 (VSS), LD3.1 (VSS), LD4.1 (VSS), LD5.1 (VSS), LD6.1 (VSS), LD7.1 (VSS), LD8.1 (VSS), LD9.1 (VSS), C10.1, C11.1, C8.1, C9.1, LD24.1 (VSS); no longer LD1.2 (VSS), LD10.2 (VSS), LD11.2 (VSS), LD12.2 (VSS), LD13.2 (VSS), LD14.2 (VSS), LD15.2 (VSS), LD16.2 (VSS), LD17.2 (VSS), LD18.2 (VSS), LD19.2 (VSS), LD2.2 (VSS), LD20.2 (VSS), LD21.2 (VSS), LD22.2 (VSS), LD23.2 (VSS), LD3.2 (VSS), LD4.2 (VSS), LD5.2 (VSS), LD6.2 (VSS), LD7.2 (VSS), LD8.2 (VSS), LD9.2 (VSS)
- net RGB: now also JP37.1 (A), LD21.2 (DIN); no longer JP37.2 (B), LD21.3 (DIN)
- net VCC: now also LD1.3 (VDD), LD10.3 (VDD), LD11.3 (VDD), LD12.3 (VDD), LD13.3 (VDD), LD14.3 (VDD), LD15.3 (VDD), LD16.3 (VDD), LD17.3 (VDD), LD18.3 (VDD), LD19.3 (VDD), LD2.3 (VDD), LD20.3 (VDD), LD21.3 (VDD), LD22.3 (VDD), LD23.3 (VDD), LD3.3 (VDD), LD4.3 (VDD), LD5.3 (VDD), LD6.3 (VDD), LD7.3 (VDD), LD8.3 (VDD), LD9.3 (VDD), C10.2, C11.2, C8.2, C9.2, LD24.3 (VDD); no longer LD1.4 (VDD), LD10.4 (VDD), LD11.4 (VDD), LD12.4 (VDD), LD13.4 (VDD), LD14.4 (VDD), LD15.4 (VDD), LD16.4 (VDD), LD17.4 (VDD), LD18.4 (VDD), LD19.4 (VDD), LD2.4 (VDD), LD20.4 (VDD), LD21.4 (VDD), LD22.4 (VDD), LD23.4 (VDD), LD3.4 (VDD), LD4.4 (VDD), LD5.4 (VDD), LD6.4 (VDD), LD7.4 (VDD), LD8.4 (VDD), LD9.4 (VDD)
- net col_1: now also SW7.2
- net col_2: now also SW11.2; no longer SW7.2
- net col_3: now also SW15.2; no longer SW11.2
- net col_4: now also SW19.2; no longer SW15.2
- net row_3: now also D19.1 (K)
- new net: JP37.2 (B), JP38.1 (A), LD21.4 (DOUT), LD22.2 (DIN)
- new net: D19.2 (A), SW19.1
- new net: LD17.2 (DIN), LD18.2 (DIN), LD19.2 (DIN), LD20.2 (DIN), LD23.4 (DOUT), LD24.2 (DIN)
- new net: LD15.2 (DIN), LD19.4 (DOUT)
- new net: LD4.2 (DIN), LD7.4 (DOUT)
- new net: JP38.2 (B), LD22.4 (DOUT), LD23.2 (DIN)
- new net: LD10.2 (DIN), LD13.4 (DOUT)
- new net: LD10.4 (DOUT), LD7.2 (DIN)
- new net: LD1.2 (DIN), LD2.2 (DIN), LD3.2 (DIN), LD6.4 (DOUT)
- new net: LD14.2 (DIN), LD18.4 (DOUT)
- new net: LD13.2 (DIN), LD17.4 (DOUT)
- new net: LD12.4 (DOUT), LD9.2 (DIN)
- new net: LD6.2 (DIN), LD9.4 (DOUT)
- new net: LD11.2 (DIN), LD14.4 (DOUT)
- new net: LD11.4 (DOUT), LD8.2 (DIN)
- new net: LD12.2 (DIN), LD15.4 (DOUT)
- new net: LD5.2 (DIN), LD8.4 (DOUT)
- new net: LD16.2 (DIN), LD20.4 (DOUT)
- no-connect marks 6 -> 7
Other:
- moved on the sheet: D11, D15, D7, JP37, JP38, LD1, LD10, LD11, LD12, LD13, LD14, LD15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
