File: pcb/KoRN.kicad_pcb (KiCad board)
At the start: 2 copper layers, 160.2 x 90.5 mm, 143 parts, among them J1 Joystick_L1, J10 OLED, J11 AudioJack4_L, J12 AudioJack4_R, J2 Joystick_L2, J3 MCU_3pin, J4 MCU_inside, J5 USB_5V, J6 Joystick_R1, J7 Joystick_R2, J8 MCU_outside, J9 Battery, SW1 SW_Push, SW10 SW_Push, SW11 SW_Push, SW12 SW_Push, SW13 SW_Push, SW14 SW_Push, SW15 SW_Push, SW16 SW_Push, SW17 SW_Push, SW18 SW_Push, SW19 SW_Push, SW2 SW_Push, SW20 SW_Push, SW21 SW_Push, SW22 SW_Push, SW3 SW_Push, SW4 SW_Push, SW5 SW_Push, SW6 SW_Push, SW7 SW_Push, SW8 SW_Push, SW9 SW_Push, U1 DRV2667

Commit message: Rename to KoRN
Parts:
- BZ1: footprint ErgoGrid:PiezoDisc_15mm_12mm -> KoRN:PiezoDisc_15mm_12mm
- H1, H2: footprint ErgoGrid:Joystick_nintendo_switch -> KoRN:Joystick_nintendo_switch
- J3: footprint ErgoGrid:ProMicro_3pin -> KoRN:ProMicro_3pin
- JP1, JP10, JP11, JP12, JP13, JP14, JP15, JP16, JP17, JP18, JP19, JP2, JP20, JP21, JP22, JP23, JP24, JP25, JP26, JP27, JP28, JP29, JP3, JP30, JP31, JP32, JP33, JP34, JP35, JP36, JP4, JP5, JP6, JP7, JP8, JP9: footprint ErgoGrid:SolderJumper -> KoRN:SolderJumper
- JP37: renamed from JP38; footprint ErgoGrid:SolderJumper -> KoRN:SolderJumper
- JP38: renamed from JP37; footprint ErgoGrid:SolderJumper -> KoRN:SolderJumper
- LD1, LD10, LD11, LD12, LD13, LD14, LD15, LD16, LD17, LD18, LD19, LD2, LD20, LD3, LD4, LD5, LD6, LD7, LD8, LD9: footprint ErgoGrid:SK6812_mini-e_rgb_reversible -> KoRN:SK6812_mini-e_rgb_reversible
- LD21: renamed from LD24; footprint ErgoGrid:SK6812_mini-e_rgb_reversible -> KoRN:SK6812_mini-e_rgb_reversible
- LD22: renamed from LD23; footprint ErgoGrid:SK6812_mini-e_rgb_reversible -> KoRN:SK6812_mini-e_rgb_reversible
- LD23: renamed from LD21; footprint ErgoGrid:SK6812_mini-e_rgb_reversible -> KoRN:SK6812_mini-e_rgb_reversible
- LD24: renamed from LD22; footprint ErgoGrid:SK6812_mini-e_rgb_reversible -> KoRN:SK6812_mini-e_rgb_reversible
- S1, S2: footprint ErgoGrid:ResetButton -> KoRN:ResetButton
Connections:
- net /key_grid/col_0 renamed /keys/col_0
- net /key_grid/col_1 renamed /keys/col_1
- net /key_grid/col_2 renamed /keys/col_2
- net /key_grid/col_3 renamed /keys/col_3
- net /key_grid/col_4 renamed /keys/col_4
- net /key_grid/col_5 renamed /keys/col_5
- net /key_grid/row_0 renamed /keys/row_0
- net /key_grid/row_1 renamed /keys/row_1
- net /key_grid/row_2 renamed /keys/row_2
- net /key_grid/row_3 renamed /keys/row_3
- J8 pad 12: /key_grid/RGB -> /keys/RGB
- JP37 pad 1: Net-(JP37-B) -> /keys/RGB
- JP37 pad 2: /key_grid/RGB -> Net-(JP37-B)
- JP38 pad 1: Net-(JP37-A) -> Net-(JP37-B)
- JP38 pad 2: Net-(JP37-B) -> Net-(JP38-B)
- LD21 pad 2: /key_grid/RGB -> /keys/RGB
- LD22 pad 4: Net-(JP37-A) -> Net-(JP38-B)
- LD23 pad 2: Net-(JP37-A) -> Net-(JP38-B)
Routing:
- net Net-(JP37-B): track 44.3 -> 79.3 mm, vias 3 -> 6
- net Net-(LD5-DIN): track 0.00 -> 26.8 mm, vias 0 -> 4
- net Net-(LD11-DOUT): track 0.00 -> 25.3 mm, vias 0 -> 3
- net Net-(LD11-DIN): track 0.00 -> 21.8 mm, vias 0 -> 3
- net Net-(LD14-DIN): track 0.00 -> 21.0 mm, vias 0 -> 3
- net /key_grid/RGB: track 20.9 -> 0.00 mm, vias 1 -> 0
- net Net-(JP37-A): track 14.1 -> 0.00 mm, vias 2 -> 0
- net VCC: track 507.0 -> 515.8 mm, vias 14 -> 17
- net JoyBtn: vias 2 -> 3
- net GND: vias 9 -> 10
- net AIN_1: vias 1 -> 2
- net AIN_0: vias 1 -> 2
