File: pcb/KoRN.kicad_sch (KiCad schematic)
At the start: 67 parts, among them J1 Joystick_L1, J10 OLED, J11 AudioJack4_L, J12 AudioJack4_R, J2 Joystick_L2, J3 MCU_3pin, J4 MCU_inside, J5 USB_5V, J6 Joystick_R1, J7 Joystick_R2, J8 MCU_outside, J9 Battery, U1 DRV2667

Commit message: Rename to KoRN
Parts:
- BZ1: footprint ErgoGrid:PiezoDisc_15mm_12mm -> KoRN:PiezoDisc_15mm_12mm
- H1, H2: footprint ErgoGrid:Joystick_nintendo_switch -> KoRN:Joystick_nintendo_switch
- J3: footprint ErgoGrid:ProMicro_3pin -> KoRN:ProMicro_3pin
- JP1, JP10, JP11, JP12, JP13, JP14, JP15, JP16, JP17, JP18, JP19, JP2, JP20, JP21, JP22, JP23, JP24, JP25, JP26, JP27, JP28, JP29, JP3, JP30, JP31, JP32, JP33, JP34, JP35, JP36, JP4, JP5, JP6, JP7, JP8, JP9: footprint ErgoGrid:SolderJumper -> KoRN:SolderJumper
- S1, S2: footprint ErgoGrid:ResetButton -> KoRN:ResetButton
- U1: symbol ErgoGrid_SymLib:DRV2667 -> KoRN:DRV2667
Other:
- sheet key_grid renamed keys
- sheet keys: file key_grid.kicad_sch -> keys.kicad_sch
