File: pcb/keys.kicad_sch (KiCad schematic)
At the start: 76 parts, among them SW1 SW_Push, SW10 SW_Push, SW11 SW_Push, SW12 SW_Push, SW13 SW_Push, SW14 SW_Push, SW15 SW_Push, SW16 SW_Push, SW17 SW_Push, SW18 SW_Push, SW19 SW_Push, SW2 SW_Push, SW20 SW_Push, SW21 SW_Push, SW22 SW_Push, SW3 SW_Push, SW4 SW_Push, SW5 SW_Push, SW6 SW_Push, SW7 SW_Push, SW8 SW_Push, SW9 SW_Push

Commit message: Rename to KoRN
Parts:
- JP37, JP38: footprint ErgoGrid:SolderJumper -> KoRN:SolderJumper
- LD1, LD10, LD11, LD12, LD13, LD14, LD15, LD16, LD17, LD18, LD19, LD2, LD20, LD21, LD22, LD23, LD24, LD3, LD4, LD5, LD6, LD7, LD8, LD9: footprint ErgoGrid:SK6812_mini-e_rgb_reversible -> KoRN:SK6812_mini-e_rgb_reversible
